File: _saved_uJTAG.sch (KiCad schematic (older format))
At the start: 29 parts, among them J1 USB_3, P1 CONN_6, U1 FT232H, U2 LD3985M, X1 CRYSTAL

Commit message: Forked the Repo, updated file types and relaid pcb.
Parts:
- U2: footprint SOT23-5 -> TO_SOT_Packages_SMD:SOT-23-5
Changed lines of the file:
@@
 F 0 "U2" H 2350 5450 60  0000 C CNN
 F 1 "LD3985M" H 2100 5900 60  0000 C CNN
-F 2 "SOT23-5" H 2000 5450 60  0000 C CNN
+F 2 "TO_SOT_Packages_SMD:SOT-23-5" H 2000 5450 60  0000 C CNN
 F 3 "" H 2100 5700 60  0001 C CNN
 	1    2100 5700
