File: uJTAG.sch (KiCad schematic (older format))
At the start: 29 parts, among them J1 USB_3, P1 CONN_6, U1 FT232H, U2 LD3985M, X1 CRYSTAL

Commit message: updated header to conform to the AVR JTAG style.
Parts:
- removed P1: CONN_6, Pin_Headers:Pin_Header_Straight_2x05, symbol CONN_6
- added P1: AVR JTAG, Pin_Headers:Pin_Header_Angled_2x05, symbol CONN_02X05
- U2: footprint SOT23-5 -> TO_SOT_Packages_SMD:SOT-23-5
Connections:
- no-connect marks 18 -> 21
Other:
- moved on the sheet: D2
